File: badger.sch (EAGLE design)
At the start: 37 parts, among them Q1 MOSFET-NCHANNEL2N7002PW, U1 NCP1402

Commit message: initial placing
Parts:
- added V3.3, VIN, VREG: TEST-POINT3X4, SparkFun-Passives:TEST-POINT3X4
Connections:
- new net V3.3: V3.3.1
- net GPIO4: now also JP3.4; no longer JP3.3
- net GPIO5: now also JP3.3; no longer JP3.4
- net VIN: now also VIN.1
- net VREG: now also VREG.1
Changed lines of the file:
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@@
 <layers>
 <layer number="1" name="Top" color="4" fill="1" visible="no" active="no"/>
+<layer number="2" name="Route2" color="1" fill="3" visible="no" active="no"/>
+<layer number="3" name="Route3" color="4" fill="3" visible="no" active="no"/>
+<layer number="14" name="Route14" color="1" fill="6" visible="no" active="no"/>
+<layer number="15" name="Route15" color="4" fill="6" visible="no" active="no"/>
 <layer number="16" name="Bottom" color="1" fill="1" visible="no" active="no"/>
 <layer number="17" name="Pads" color="2" fill="1" visible="no" active="no"/>
@@
 <part name="GND14" library="SparkFun" deviceset="GND" device=""/>
 <part name="U$3" library="adafruit" deviceset="PS603" device="SPK"/>
+<part name="VIN" library="SparkFun-Passives" deviceset="TEST-POINT" device="3X4"/>
+<part name="VREG" library="SparkFun-Passives" deviceset="TEST-POINT" device="3X4"/>
+<part name="V3.3" library="SparkFun-Passives" deviceset="TEST-POINT" device="3X4"/>
 </parts>
 <sheets>
@@
 <instance part="GND14" gate="1" x="-83.82" y="35.56"/>
 <instance part="U$3" gate="G$1" x="-83.82" y="60.96" rot="R90"/>
+<instance part="VIN" gate="G$1" x="-119.38" y="-20.32"/>
+<instance part="VREG" gate="G$1" x="-119.38" y="-30.48"/>
+<instance part="V3.3" gate="G$1" x="-119.38" y="-40.64"/>
 </instances>
 <busses>
@@
 <label x="-91.44" y="76.2" size="1.778" layer="95"/>
 </segment>
+<segment>
+<pinref part="VIN" gate="G$1" pin="1"/>
+<wire x1="-119.38" y1="-20.32" x2="-129.54" y2="-20.32" width="0.1524" layer="91"/>
+<label x="-129.54" y="-20.32" size="1.778" layer="95"/>
+</segment>
 </net>
 <net name="RESET" class="0">
@@
 </segment>
 <segment>
+<pinref part="CHEAPO-3" gate="G$1" pin="3"/>
+<wire x1="-66.04" y1="-2.54" x2="-58.42" y2="-2.54" width="0.1524" layer="91"/>
+<label x="-66.04" y="-2.54" size="1.778" layer="95"/>
+</segment>
+<segment>
+<pinref part="JP3" gate="G$1" pin="3"/>
+<wire x1="134.62" y1="-7.62" x2="124.46" y2="-7.62" width="0.1524" layer="91"/>
+<label x="124.46" y="-7.62" size="1.778" layer="95"/>
+</segment>
+</net>
+<net name="GPIO4" class="0">
+<segment>
+<pinref part="U2" gate="G$1" pin="GPIO4"/>
+<wire x1="160.02" y1="63.5" x2="167.64" y2="63.5" width="0.1524" layer="91"/>
+<label x="162.56" y="63.5" size="1.778" layer="95"/>
+</segment>
+<segment>
+<pinref part="CHEAPO-2" gate="G$1" pin="3"/>
+<wire x1="-50.8" y1="5.08" x2="-40.64" y2="5.08" width="0.1524" layer="91"/>
+<label x="-45.72" y="5.08" size="1.778" layer="95"/>
+</segment>
+<segment>
 <pinref part="JP3" gate="G$1" pin="4"/>
 <wire x1="134.62" y1="-10.16" x2="124.46" y2="-10.16" width="0.1524" layer="91"/>
 <label x="124.46" y="-10.16" size="1.778" layer="95"/>
-</segment>
-<segment>
-<pinref part="CHEAPO-3" gate="G$1" pin="3"/>
-<wire x1="-66.04" y1="-2.54" x2="-58.42" y2="-2.54" width="0.1524" layer="91"/>
-<label x="-66.04" y="-2.54" size="1.778" layer="95"/>
-</segment>
-</net>
-<net name="GPIO4" class="0">
-<segment>
-<pinref part="U2" gate="G$1" pin="GPIO4"/>
-<wire x1="160.02" y1="63.5" x2="167.64" y2="63.5" width="0.1524" layer="91"/>
-<label x="162.56" y="63.5" size="1.778" layer="95"/>
-</segment>
-<segment>
-<pinref part="JP3" gate="G$1" pin="3"/>
-<wire x1="134.62" y1="-7.62" x2="124.46" y2="-7.62" width="0.1524" layer="91"/>
-<label x="124.46" y="-7.62" size="1.778" layer="95"/>
-</segment>
-<segment>
-<pinref part="CHEAPO-2" gate="G$1" pin="3"/>
-<wire x1="-50.8" y1="5.08" x2="-40.64" y2="5.08" width="0.1524" layer="91"/>
-<label x="-45.72" y="5.08" size="1.778" layer="95"/>
 </segment>
 </net>
@@
 <label x="55.88" y="0" size="1.778" layer="95"/>
 </segment>
+<segment>
+<pinref part="VREG" gate="G$1" pin="1"/>
+<wire x1="-119.38" y1="-30.48" x2="-129.54" y2="-30.48" width="0.1524" layer="91"/>
+<label x="-129.54" y="-30.48" size="1.778" layer="95"/>
+</segment>
 </net>
 <net name="VFTDI" class="0">
@@
 </segment>
 </net>
+<net name="V3.3" class="0">
+<segment>
+<pinref part="V3.3" gate="G$1" pin="1"/>
+<wire x1="-119.38" y1="-40.64" x2="-129.54" y2="-40.64" width="0.1524" layer="91"/>
+<label x="-129.54" y="-40.64" size="1.778" layer="95"/>
+</segment>
+</net>

Commit message: as sent to itead
Parts:
- added C3: 10uF, SparkFun-Capacitors:10UF-6.3V-20%(0603)
- added R2, R3, R4: 10K, SparkFun-Resistors:10KOHM-1/10W-1%(0603)0603
- R1: value (none) -> 10K; device SparkFun-Resistors:RESISTOR-ARRAY0603-ARV -> SparkFun-Resistors:10KOHM-1/10W-1%(0603)0603
Connections:
- removed net V3.3: V3.3.1
- net 3.3V: now also C3.1, R1.2, R2.2, R3.2, V3.3.1; no longer R1A.1, R1D.2, R1R.1
- net CH_PD: now also R1.1; no longer R1D.1
- net GND: now also C3.2, R4.1; no longer R1B.2
- net GPIO0: now also R3.1; no longer R1A.2
- net GPIO2: now also R2.1; no longer R1R.2
- net N$1: now also R4.2; no longer R1B.1
Changed lines of the file:
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@@
 <part name="U2" library="esp8266modules" deviceset="ESP12E" device="SMD"/>
 <part name="GND5" library="SparkFun" deviceset="GND" device=""/>
-<part name="R1" library="SparkFun-Resistors" deviceset="RESISTOR-ARRAY" device="0603-ARV"/>
 <part name="SUPPLY2" library="SparkFun-Aesthetics" deviceset="3.3V" device=""/>
 <part name="SUPPLY3" library="SparkFun-Aesthetics" deviceset="3.3V" device=""/>
@@
 <part name="VREG" library="SparkFun-Passives" deviceset="TEST-POINT" device="3X4"/>
 <part name="V3.3" library="SparkFun-Passives" deviceset="TEST-POINT" device="3X4"/>
+<part name="SUPPLY6" library="SparkFun-Aesthetics" deviceset="3.3V" device=""/>
+<part name="C3" library="SparkFun-Capacitors" deviceset="10UF-6.3V-20%(0603)" device="" value="10uF"/>
+<part name="GND15" library="SparkFun" deviceset="GND" device=""/>
+<part name="SUPPLY7" library="SparkFun-Aesthetics" deviceset="3.3V" device=""/>
+<part name="R1" library="SparkFun-Resistors" deviceset="10KOHM-1/10W-1%(0603)" device="0603" value="10K"/>
+<part name="R2" library="SparkFun-Resistors" deviceset="10KOHM-1/10W-1%(0603)" device="0603" value="10K"/>
+<part name="R3" library="SparkFun-Resistors" deviceset="10KOHM-1/10W-1%(0603)" device="0603" value="10K"/>
+<part name="R4" library="SparkFun-Resistors" deviceset="10KOHM-1/10W-1%(0603)" device="0603" value="10K"/>
 </parts>
 <sheets>
@@
 <instance part="U2" gate="G$1" x="144.78" y="60.96"/>
 <instance part="GND5" gate="1" x="177.8" y="27.94"/>
-<instance part="R1" gate="A" x="205.74" y="68.58" rot="R270"/>
-<instance part="R1" gate="B" x="109.22" y="15.24" rot="R270"/>
-<instance part="R1" gate="R" x="177.8" y="68.58" rot="R270"/>
-<instance part="R1" gate="D" x="101.6" y="76.2" rot="R90"/>
 <instance part="SUPPLY2" gate="G$1" x="101.6" y="83.82"/>
 <instance part="SUPPLY3" gate="G$1" x="177.8" y="83.82"/>
@@
 <instance part="VREG" gate="G$1" x="-119.38" y="-30.48"/>
 <instance part="V3.3" gate="G$1" x="-119.38" y="-40.64"/>
+<instance part="SUPPLY6" gate="G$1" x="-134.62" y="-38.1"/>
+<instance part="C3" gate="G$1" x="142.24" y="86.36"/>
+<instance part="GND15" gate="1" x="142.24" y="78.74"/>
+<instance part="SUPPLY7" gate="G$1" x="142.24" y="93.98"/>
+<instance part="R1" gate="G$1" x="101.6" y="76.2" rot="R90"/>
+<instance part="R2" gate="G$1" x="177.8" y="68.58" rot="R90"/>
+<instance part="R3" gate="G$1" x="205.74" y="68.58" rot="R90"/>
+<instance part="R4" gate="G$1" x="109.22" y="15.24" rot="R90"/>
 </instances>
 <busses>
@@
 </segment>
 <segment>
-<pinref part="R1" gate="B" pin="2"/>
 <pinref part="GND9" gate="1" pin="GND"/>
 <wire x1="109.22" y1="10.16" x2="109.22" y2="7.62" width="0.1524" layer="91"/>
+<pinref part="R4" gate="G$1" pin="1"/>
 </segment>
 <segment>
@@
 <pinref part="GND14" gate="1" pin="GND"/>
 <wire x1="-83.82" y1="43.18" x2="-83.82" y2="38.1" width="0.1524" layer="91"/>
+</segment>
+<segment>
+<pinref part="GND15" gate="1" pin="GND"/>
+<pinref part="C3" gate="G$1" pin="2"/>
+<wire x1="142.24" y1="81.28" x2="142.24" y2="83.82" width="0.1524" layer="91"/>
 </segment>
 </net>
@@
 </segment>
 <segment>
-<pinref part="R1" gate="A" pin="2"/>
 <wire x1="205.74" y1="63.5" x2="205.74" y2="58.42" width="0.1524" layer="91"/>
 <wire x1="205.74" y1="58.42" x2="195.58" y2="58.42" width="0.1524" layer="91"/>
@@
 <wire x1="205.74" y1="58.42" x2="205.74" y2="55.88" width="0.1524" layer="91"/>
 <junction x="205.74" y="58.42"/>
+<pinref part="R3" gate="G$1" pin="1"/>
 </segment>
 <segment>
@@
 <segment>
 <pinref part="SUPPLY2" gate="G$1" pin="3.3V"/>
-<pinref part="R1" gate="D" pin="2"/>
 <wire x1="101.6" y1="83.82" x2="101.6" y2="81.28" width="0.1524" layer="91"/>
+<pinref part="R1" gate="G$1" pin="2"/>
 </segment>
 <segment>
 <pinref part="SUPPLY4" gate="G$1" pin="3.3V"/>
-<pinref part="R1" gate="A" pin="1"/>
 <wire x1="205.74" y1="76.2" x2="205.74" y2="73.66" width="0.1524" layer="91"/>
-</segment>
-<segment>
-<pinref part="R1" gate="R" pin="1"/>
+<pinref part="R3" gate="G$1" pin="2"/>
+</segment>
+<segment>
 <pinref part="SUPPLY3" gate="G$1" pin="3.3V"/>
 <wire x1="177.8" y1="73.66" x2="177.8" y2="83.82" width="0.1524" layer="91"/>
+<pinref part="R2" gate="G$1" pin="2"/>
 </segment>
 <segment>
@@
 <wire x1="20.32" y1="-10.16" x2="20.32" y2="-15.24" width="0.1524" layer="91"/>
 </segment>
+<segment>
+<pinref part="SUPPLY6" gate="G$1" pin="3.3V"/>
+<wire x1="-134.62" y1="-38.1" x2="-134.62" y2="-40.64" width="0.1524" layer="91"/>
+<pinref part="V3.3" gate="G$1" pin="1"/>
+<wire x1="-119.38" y1="-40.64" x2="-134.62" y2="-40.64" width="0.1524" layer="91"/>
+<label x="-129.54" y="-40.64" size="1.778" layer="95"/>
+</segment>
+<segment>
+<pinref part="SUPPLY7" gate="G$1" pin="3.3V"/>
+<pinref part="C3" gate="G$1" pin="1"/>
+<wire x1="142.24" y1="93.98" x2="142.24" y2="91.44" width="0.1524" layer="91"/>
+</segment>
 </net>
 <net name="CH_PD" class="0">
@@
 <pinref part="U2" gate="G$1" pin="CH_PD"/>
 <wire x1="101.6" y1="63.5" x2="127" y2="63.5" width="0.1524" layer="91"/>
-<pinref part="R1" gate="D" pin="1"/>
 <wire x1="101.6" y1="63.5" x2="101.6" y2="71.12" width="0.1524" layer="91"/>
 <label x="116.84" y="63.5" size="1.778" layer="95"/>
+<pinref part="R1" gate="G$1" pin="1"/>
 </segment>
 <segment>
@@
 <pinref part="U2" gate="G$1" pin="GPIO2"/>
 <wire x1="177.8" y1="55.88" x2="160.02" y2="55.88" width="0.1524" layer="91"/>
-<pinref part="R1" gate="R" pin="2"/>
 <wire x1="177.8" y1="55.88" x2="177.8" y2="63.5" width="0.1524" layer="91"/>
 <label x="162.56" y="55.88" size="1.778" layer="95"/>
+<pinref part="R2" gate="G$1" pin="1"/>
 </segment>
 </net>
@@
 <pinref part="GPIO15&lt;-&gt;GND" gate="1" pin="2"/>
 <wire x1="104.14" y1="25.4" x2="109.22" y2="25.4" width="0.1524" layer="91"/>
-<pinref part="R1" gate="B" pin="1"/>
 <wire x1="109.22" y1="25.4" x2="109.22" y2="20.32" width="0.1524" layer="91"/>
+<pinref part="R4" gate="G$1" pin="2"/>
 </segment>
 </net>
@@
 </segment>
 </net>
-<net name="V3.3" class="0">
-<segment>
-<pinref part="V3.3" gate="G$1" pin="1"/>
-<wire x1="-119.38" y1="-40.64" x2="-129.54" y2="-40.64" width="0.1524" layer="91"/>
-<label x="-129.54" y="-40.64" size="1.778" layer="95"/>
-</segment>
-</net>
