File: badger.sch (EAGLE design)
At the start: 46 parts, among them Q1 2N7002PW, U1 NCP1402

Commit message: Another test-spin
Signed-off-by: Hacker, J.R <r00tkillah@gmail.com>
Parts:
- removed Q1: 2N7002PW, SparkFun-DiscreteSemi:MOSFET-NCHANNEL2N7002PW
- GPIO16<->RESET: value SOLDERJUMPERTRACE -> SOLDERJUMPERNO; device SparkFun-Retired:SOLDERJUMPERTRACE -> SparkFun-Retired:SOLDERJUMPERNO
Connections:
- removed net N$18: D7.C, Q1.S, U$3.1
- net GND: now also U$3.1; no longer Q1.D
- net GPIO15: no longer Q1.G
- net GPIO16: now also CHEAPO-2.3
- net GPIO4: now also U$3.2; no longer CHEAPO-2.3
- net VIN: no longer U$3.2
Other:
- moved on the sheet: D7, U$3
Changed lines of the file:
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@@
 <setting verticaltext="up"/>
 </settings>
-<grid distance="0.1" unitdist="inch" unit="inch" style="lines" multiple="1" display="no" altdistance="0.01" altunitdist="inch" altunit="inch"/>
+<grid distance="0.025" unitdist="inch" unit="inch" style="lines" multiple="1" display="no" altdistance="0.01" altunitdist="inch" altunit="inch"/>
 <layers>
 <layer number="1" name="Top" color="4" fill="1" visible="no" active="no"/>
@@
 <part name="GND1" library="SparkFun" deviceset="GND" device=""/>
 <part name="GND6" library="SparkFun" deviceset="GND" device=""/>
-<part name="GPIO16&lt;-&gt;RESET" library="SparkFun-Retired" deviceset="SOLDERJUMPER" device="TRACE"/>
 <part name="GPIO15&lt;-&gt;GND" library="SparkFun-Retired" deviceset="SOLDERJUMPER" device="TRACE"/>
 <part name="D2" library="SparkFun-LED" deviceset="LED" device="-3MM-NO_SILK"/>
@@
 <part name="CHEAPO-3" library="SparkFun-Retired" deviceset="SOLDERJUMPER_2WAY" device="T"/>
 <part name="CHEAPO-7" library="SparkFun-Retired" deviceset="SOLDERJUMPER_2WAY" device="T"/>
-<part name="Q1" library="SparkFun-DiscreteSemi" deviceset="MOSFET-NCHANNEL" device="2N7002PW" value="2N7002PW"/>
 <part name="GND14" library="SparkFun" deviceset="GND" device=""/>
 <part name="U$3" library="adafruit" deviceset="PS603" device="SPK"/>
@@
 <part name="D7" library="SparkFun-DiscreteSemi" deviceset="DIODE" device="BAS16" value="250mA/100V"/>
 <part name="LOGO1" library="SparkFun-Aesthetics" deviceset="OSHW-LOGO" device="L-COPPER"/>
+<part name="GPIO16&lt;-&gt;RESET" library="SparkFun-Retired" deviceset="SOLDERJUMPER" device="NO"/>
 </parts>
 <sheets>
@@
 <instance part="GND1" gate="1" x="205.74" y="35.56"/>
 <instance part="GND6" gate="1" x="119.38" y="81.28"/>
-<instance part="GPIO16&lt;-&gt;RESET" gate="1" x="99.06" y="38.1"/>
 <instance part="GPIO15&lt;-&gt;GND" gate="1" x="99.06" y="25.4"/>
 <instance part="D2" gate="G$1" x="-66.04" y="-27.94"/>
@@
 <attribute name="VALUE" x="-84.455" y="5.08" size="1.778" layer="96" rot="R90"/>
 </instance>
-<instance part="Q1" gate="G$1" x="-83.82" y="43.18" rot="R180"/>
 <instance part="GND14" gate="1" x="-83.82" y="30.48"/>
-<instance part="U$3" gate="G$1" x="-83.82" y="60.96" rot="R90"/>
+<instance part="U$3" gate="G$1" x="-83.82" y="48.26" rot="R90"/>
 <instance part="VIN" gate="G$1" x="-119.38" y="-20.32"/>
 <instance part="VREG" gate="G$1" x="-119.38" y="-30.48"/>
@@
 <instance part="JP2" gate="G$1" x="185.42" y="-35.56" rot="R180"/>
 <instance part="GND16" gate="1" x="5.08" y="33.02"/>
-<instance part="D7" gate="G$1" x="-97.79" y="43.18" rot="R90"/>
+<instance part="D7" gate="G$1" x="-71.12" y="43.815" rot="R90"/>
 <instance part="LOGO1" gate="G$1" x="-22.86" y="-30.48"/>
+<instance part="GPIO16&lt;-&gt;RESET" gate="1" x="99.06" y="38.1"/>
 </instances>
 <busses>
@@
 </segment>
 <segment>
-<pinref part="Q1" gate="G$1" pin="D"/>
-<pinref part="GND14" gate="1" pin="GND"/>
-<wire x1="-83.82" y1="38.1" x2="-83.82" y2="36.83" width="0.1524" layer="91"/>
-<pinref part="D7" gate="G$1" pin="A"/>
-<wire x1="-83.82" y1="36.83" x2="-83.82" y2="33.02" width="0.1524" layer="91"/>
-<wire x1="-97.79" y1="40.64" x2="-97.79" y2="36.83" width="0.1524" layer="91"/>
-<wire x1="-97.79" y1="36.83" x2="-83.82" y2="36.83" width="0.1524" layer="91"/>
-<junction x="-83.82" y="36.83"/>
-</segment>
-<segment>
 <pinref part="GND15" gate="1" pin="GND"/>
 <pinref part="C3" gate="G$1" pin="2"/>
@@
 <wire x1="20.32" y1="-7.62" x2="7.62" y2="-7.62" width="0.1524" layer="91"/>
 <wire x1="7.62" y1="-7.62" x2="7.62" y2="-12.7" width="0.1524" layer="91"/>
+</segment>
+<segment>
+<pinref part="U$3" gate="G$1" pin="1"/>
+<pinref part="GND14" gate="1" pin="GND"/>
+<wire x1="-83.82" y1="43.18" x2="-83.82" y2="37.465" width="0.1524" layer="91"/>
+<pinref part="D7" gate="G$1" pin="A"/>
+<wire x1="-83.82" y1="37.465" x2="-83.82" y2="33.02" width="0.1524" layer="91"/>
+<wire x1="-71.12" y1="41.275" x2="-71.12" y2="37.465" width="0.1524" layer="91"/>
+<wire x1="-71.12" y1="37.465" x2="-83.82" y2="37.465" width="0.1524" layer="91"/>
+<junction x="-83.82" y="37.465"/>
 </segment>
 </net>
@@
 </segment>
 <segment>
-<pinref part="U$3" gate="G$1" pin="2"/>
-<wire x1="-83.82" y1="66.04" x2="-83.82" y2="76.2" width="0.1524" layer="91"/>
-<wire x1="-83.82" y1="76.2" x2="-93.98" y2="76.2" width="0.1524" layer="91"/>
-<label x="-91.44" y="76.2" size="1.778" layer="95"/>
-</segment>
-<segment>
 <pinref part="VIN" gate="G$1" pin="1"/>
 <wire x1="-119.38" y1="-20.32" x2="-129.54" y2="-20.32" width="0.1524" layer="91"/>
@@
 </segment>
 <segment>
-<pinref part="GPIO16&lt;-&gt;RESET" gate="1" pin="1"/>
 <wire x1="93.98" y1="38.1" x2="83.82" y2="38.1" width="0.1524" layer="91"/>
 <label x="83.82" y="38.1" size="1.778" layer="95"/>
+<pinref part="GPIO16&lt;-&gt;RESET" gate="1" pin="1"/>
 </segment>
 <segment>
@@
 </segment>
 <segment>
-<pinref part="CHEAPO-2" gate="G$1" pin="3"/>
-<wire x1="-50.8" y1="5.08" x2="-40.64" y2="5.08" width="0.1524" layer="91"/>
-<label x="-45.72" y="5.08" size="1.778" layer="95"/>
-</segment>
-<segment>
 <pinref part="JP6" gate="G$1" pin="4"/>
 <wire x1="134.62" y1="-40.64" x2="124.46" y2="-40.64" width="0.1524" layer="91"/>
 <label x="124.46" y="-40.64" size="1.778" layer="95"/>
+</segment>
+<segment>
+<pinref part="U$3" gate="G$1" pin="2"/>
+<wire x1="-83.82" y1="53.34" x2="-83.82" y2="58.42" width="0.1524" layer="91"/>
+<wire x1="-83.82" y1="58.42" x2="-83.82" y2="66.04" width="0.1524" layer="91"/>
+<wire x1="-83.82" y1="66.04" x2="-73.66" y2="66.04" width="0.1524" layer="91"/>
+<wire x1="-83.82" y1="58.42" x2="-71.12" y2="58.42" width="0.1524" layer="91"/>
+<wire x1="-71.12" y1="58.42" x2="-71.12" y2="46.355" width="0.1524" layer="91"/>
+<junction x="-83.82" y="58.42"/>
+<label x="-78.74" y="66.04" size="1.778" layer="95"/>
 </segment>
 </net>
@@
 </segment>
 <segment>
-<pinref part="GPIO16&lt;-&gt;RESET" gate="1" pin="2"/>
 <wire x1="104.14" y1="38.1" x2="114.3" y2="38.1" width="0.1524" layer="91"/>
 <label x="109.22" y="38.1" size="1.778" layer="95"/>
+<pinref part="GPIO16&lt;-&gt;RESET" gate="1" pin="2"/>
 </segment>
 <segment>
@@
 <wire x1="99.06" y1="-40.64" x2="109.22" y2="-40.64" width="0.1524" layer="91"/>
 <label x="104.14" y="-40.64" size="1.778" layer="95"/>
+</segment>
+<segment>
+<pinref part="CHEAPO-2" gate="G$1" pin="3"/>
+<wire x1="-50.8" y1="5.08" x2="-37.465" y2="5.08" width="0.1524" layer="91"/>
+<label x="-44.45" y="5.08" size="1.778" layer="95"/>
 </segment>
 </net>
@@
 <wire x1="134.62" y1="-48.26" x2="124.46" y2="-48.26" width="0.1524" layer="91"/>
 <label x="124.46" y="-48.26" size="1.778" layer="95"/>
-</segment>
-<segment>
-<pinref part="Q1" gate="G$1" pin="G"/>
-<wire x1="-76.2" y1="43.18" x2="-63.5" y2="43.18" width="0.1524" layer="91"/>
-<label x="-71.12" y="43.18" size="1.778" layer="95"/>
 </segment>
 </net>
@@
 </segment>
 </net>
-<net name="N$18" class="0">
-<segment>
-<pinref part="U$3" gate="G$1" pin="1"/>
-<pinref part="Q1" gate="G$1" pin="S"/>
-<wire x1="-83.82" y1="55.88" x2="-83.82" y2="52.07" width="0.1524" layer="91"/>
-<pinref part="D7" gate="G$1" pin="C"/>
-<wire x1="-83.82" y1="52.07" x2="-83.82" y2="48.26" width="0.1524" layer="91"/>
-<wire x1="-83.82" y1="52.07" x2="-97.79" y2="52.07" width="0.1524" layer="91"/>
-<wire x1="-97.79" y1="52.07" x2="-97.79" y2="45.72" width="0.1524" layer="91"/>
-<junction x="-83.82" y="52.07"/>
-</segment>
-</net>

Commit message: reconnect diode; via cleanups
Noticed that stapling vias were octogon and larger drill diameter.  Fixed

Signed-off-by: Hacker, J.R <r00tkillah@gmail.com>
Connections:
- net GPIO4: now also D7.C
Changed lines of the file:
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@@
 <junction x="-83.82" y="58.42"/>
 <label x="-78.74" y="66.04" size="1.778" layer="95"/>
+<pinref part="D7" gate="G$1" pin="C"/>
 </segment>
 </net>
