File: badger.brd (EAGLE design)
At the start: 149.2 x 68.3 mm, 46 parts, among them Q1 2N7002PW, U1 NCP1402

Commit message: final(?) design? - rerouted - rgb led now with common gnd - rgb led now powered by vin with cheapo varient - new cam
Connections:
- net 3.3V: no longer D5.C
- net GND: now also D5.C; no longer CHEAPO-4.3, CHEAPO-5.3, CHEAPO-6.3
- net GPIO15: now also Q1.1
- net GPIO16: no longer Q1.1
- net VIN: now also CHEAPO-4.3, CHEAPO-5.3, CHEAPO-6.3
Routing:
- net GPIO15: track 42.2 -> 124.4 mm, vias 0 -> 2
- net VIN: track 129.5 -> 206.2 mm
- net GPIO16: track 115.7 -> 56.2 mm, vias 4 -> 2
- net 3.3V: track 115.2 -> 68.1 mm, vias 4 -> 2
- net RESET: track 62.7 -> 73.1 mm, vias 3 -> 2
- net RX: track 47.5 -> 56.8 mm
- net VFTDI: track 24.3 -> 18.4 mm
- net GPIO0: track 73.1 -> 78.3 mm, vias 2 -> 1
- net N$5: track 96.5 -> 101.4 mm, vias 2 -> 4
- net GPIO13: track 40.4 -> 43.8 mm
- net GPIO5: track 51.0 -> 52.8 mm
- net TX: track 60.3 -> 59.1 mm, vias 0 -> 2
- net N$16: track 9.75 -> 10.6 mm
- net GPIO12: track 36.9 -> 37.7 mm, vias 3 -> 2
- net N$7: track 27.4 -> 26.7 mm
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
Commit message: reapply design rules; dimension/pour 6mil; gnd
added gnd trace near antenna in case of mill problems

Signed-off-by: Hacker, J.R <r00tkillah@gmail.com>
Routing:
- net GND: track 0.00 -> 14.9 mm, vias 29 -> 38
- net TX: track 59.1 -> 60.6 mm
Changed lines of the file:
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@@
 </class>
 </classes>
-<designrules name="default *">
+<designrules name="oshpark-2layer *">
 <description language="de">&lt;b&gt;EAGLE Design Rules&lt;/b&gt;
 &lt;p&gt;
@@
 Einstellungen hier und speichern die Design Rules unter
 einem neuen Namen ab.</description>
-<description language="en">&lt;b&gt;EAGLE Design Rules&lt;/b&gt;
+<description language="en">&lt;b&gt;Laen's PCB Order Design Rules&lt;/b&gt;
 &lt;p&gt;
-The default Design Rules have been set to cover
-a wide range of applications. Your particular design
-may have different requirements, so please make the
-necessary adjustments and save your customized
-design rules under a new name.</description>
+Please make sure your boards conform to these design rules.</description>
 <param name="layerSetup" value="(1*16)"/>
-<param name="mtCopper" value="0.035mm 0.035mm 0.035mm 0.035mm 0.035mm 0.035mm 0.035mm 0.035mm 0.035mm 0.035mm 0.035mm 0.035mm 0.035mm 0.035mm 0.035mm 0.035mm"/>
-<param name="mtIsolate" value="1.5mm 0.15mm 0.2mm 0.15mm 0.2mm 0.15mm 0.2mm 0.15mm 0.2mm 0.15mm 0.2mm 0.15mm 0.2mm 0.15mm 0.2mm"/>
-<param name="mdWireWire" value="8mil"/>
-<param name="mdWirePad" value="8mil"/>
-<param name="mdWireVia" value="8mil"/>
-<param name="mdPadPad" value="8mil"/>
-<param name="mdPadVia" value="8mil"/>
-<param name="mdViaVia" value="8mil"/>
-<param name="mdSmdPad" value="8mil"/>
-<param name="mdSmdVia" value="8mil"/>
-<param name="mdSmdSmd" value="8mil"/>
+<param name="mtCopper" value="0.0356mm 0.0356mm 0.0356mm 0.0356mm 0.0356mm 0.0356mm 0.0356mm 0.0356mm 0.0356mm 0.0356mm 0.0356mm 0.0356mm 0.0356mm 0.0356mm 0.0356mm 0.0356mm"/>
+<param name="mtIsolate" value="1.5011mm 0.1499mm 0.2007mm 0.1499mm 0.2007mm 0.1499mm 0.2007mm 0.1499mm 0.2007mm 0.1499mm 0.2007mm 0.1499mm 0.2007mm 0.1499mm 0.2007mm"/>
+<param name="mdWireWire" value="6mil"/>
+<param name="mdWirePad" value="6mil"/>
+<param name="mdWireVia" value="6mil"/>
+<param name="mdPadPad" value="6mil"/>
+<param name="mdPadVia" value="6mil"/>
+<param name="mdViaVia" value="6mil"/>
+<param name="mdSmdPad" value="6mil"/>
+<param name="mdSmdVia" value="6mil"/>
+<param name="mdSmdSmd" value="6mil"/>
 <param name="mdViaViaSameLayer" value="8mil"/>
 <param name="mnLayersViaInSmd" value="2"/>
-<param name="mdCopperDimension" value="5mil"/>
-<param name="mdDrill" value="8mil"/>
+<param name="mdCopperDimension" value="6mil"/>
+<param name="mdDrill" value="6mil"/>
 <param name="mdSmdStop" value="0mil"/>
-<param name="msWidth" value="10mil"/>
-<param name="msDrill" value="24mil"/>
-<param name="msMicroVia" value="9.99mm"/>
+<param name="msWidth" value="6mil"/>
+<param name="msDrill" value="13mil"/>
+<param name="msMicroVia" value="13mil"/>
 <param name="msBlindViaRatio" value="0.5"/>
 <param name="rvPadTop" value="0.25"/>
@@
 <param name="rvMicroViaOuter" value="0.25"/>
 <param name="rvMicroViaInner" value="0.25"/>
-<param name="rlMinPadTop" value="10mil"/>
+<param name="rlMinPadTop" value="7mil"/>
 <param name="rlMaxPadTop" value="20mil"/>
-<param name="rlMinPadInner" value="10mil"/>
+<param name="rlMinPadInner" value="7mil"/>
 <param name="rlMaxPadInner" value="20mil"/>
-<param name="rlMinPadBottom" value="10mil"/>
+<param name="rlMinPadBottom" value="7mil"/>
 <param name="rlMaxPadBottom" value="20mil"/>
-<param name="rlMinViaOuter" value="8mil"/>
+<param name="rlMinViaOuter" value="7mil"/>
 <param name="rlMaxViaOuter" value="20mil"/>
-<param name="rlMinViaInner" value="8mil"/>
+<param name="rlMinViaInner" value="7mil"/>
 <param name="rlMaxViaInner" value="20mil"/>
 <param name="rlMinMicroViaOuter" value="4mil"/>
@@
 <contactref element="JP1" pad="6"/>
 <contactref element="D5" pad="C"/>
-<via x="87.952175" y="59.433028125" extent="1-16" drill="0.6"/>
+<via x="88.46015" y="59.14275625" extent="1-16" drill="0.6"/>
 <via x="37.6626875" y="61.1020875" extent="1-16" drill="0.6"/>
 <via x="81.783909375" y="61.6100625" extent="1-16" drill="0.6"/>
@@
 <via x="115.890778125" y="54.570984375" extent="1-16" drill="0.6"/>
 <via x="115.890778125" y="46.7336625" extent="1-16" drill="0.6"/>
+<via x="91.798265625" y="27.866034375" extent="1-16" drill="0.6"/>
+<via x="92.814215625" y="22.0606125" extent="1-16" drill="0.6"/>
+<via x="90.056640625" y="18.57735625" extent="1-16" drill="0.6"/>
+<via x="89.76636875" y="15.021534375" extent="1-16" drill="0.6"/>
+<wire x1="94.99125" y1="63.714528125" x2="97.095715625" y2="64.0048" width="0.4064" layer="16"/>
+<wire x1="97.095715625" y1="64.0048" x2="98.619640625" y2="64.222503125" width="0.4064" layer="16"/>
+<wire x1="98.619640625" y1="64.222503125" x2="99.925859375" y2="64.512775" width="0.4064" layer="16"/>
+<wire x1="99.925859375" y1="64.512775" x2="101.885190625" y2="64.44020625" width="0.4064" layer="16"/>
+<wire x1="101.885190625" y1="64.44020625" x2="103.11884375" y2="64.44020625" width="0.4064" layer="16"/>
+<wire x1="107.110071875" y1="59.941003125" x2="107.110071875" y2="59.505596875" width="0.3048" layer="16"/>
+<wire x1="107.110071875" y1="59.505596875" x2="105.295875" y2="59.578165625" width="0.3048" layer="16"/>
+<wire x1="105.295875" y1="59.578165625" x2="105.295875" y2="56.457746875" width="0.3048" layer="16"/>
+<wire x1="105.295875" y1="56.457746875" x2="103.98965625" y2="56.167478125" width="0.3048" layer="16"/>
+<via x="103.98965625" y="56.167478125" extent="1-16" drill="0.6"/>
+<via x="107.182640625" y="60.013571875" extent="1-16" drill="0.6"/>
+<via x="95.57179375" y="54.716121875" extent="1-16" drill="0.6"/>
+<via x="98.32936875" y="49.2735375" extent="1-16" drill="0.6"/>
+<via x="91.65313125" y="48.475290625" extent="1-16" drill="0.6"/>
 </signal>
 <signal name="VIN">
@@
 <wire x1="86.0425" y1="54.76875" x2="86.0425" y2="58.7375" width="0.254" layer="1"/>
 <wire x1="90.32875" y1="54.76875" x2="86.0425" y2="54.76875" width="0.254" layer="16"/>
-<wire x1="105.7275" y1="54.76875" x2="90.32875" y2="54.76875" width="0.254" layer="1"/>
 <wire x1="105.7275" y1="61.9125" x2="105.7275" y2="54.76875" width="0.254" layer="1"/>
 <wire x1="68.42125" y1="48.895" x2="68.41963125" y2="48.814790625" width="0.254" layer="1"/>
@@
 <via x="86.0425" y="54.76875" extent="1-16" drill="0.6096"/>
 <via x="90.32875" y="54.76875" extent="1-16" drill="0.6096"/>
+<wire x1="105.7275" y1="54.76875" x2="102.08295625" y2="54.76875" width="0.3048" layer="1"/>
+<wire x1="102.08295625" y1="54.76875" x2="100.2887" y2="52.97449375" width="0.3048" layer="1"/>
+<wire x1="100.2887" y1="52.97449375" x2="92.12300625" y2="52.97449375" width="0.3048" layer="1"/>
+<wire x1="92.12300625" y1="52.97449375" x2="90.32875" y2="54.76875" width="0.3048" layer="1"/>
 </signal>
 <signal name="3.3V">

Commit message: Another test-spin
Signed-off-by: Hacker, J.R <r00tkillah@gmail.com>
Parts:
- removed Q1: 2N7002PW, SparkFun-DiscreteSemi:SOT323
- GPIO16<->RESET: value SOLDERJUMPERTRACE -> SOLDERJUMPERNO; device SparkFun-Retired:SJ_2S-TRACE -> SparkFun-Retired:SJ_2S-NO
- moved GPIO16<->RESET 48.2 mm to (81.9, 20.3), turned to 180 degrees
- moved D7 3.98 mm to (36.4, 21.5), turned to 0 degrees
- moved R4 1.62 mm to (116.4, 64.4), turned to 270 degrees
Connections:
- removed net N$18: D7.C, Q1.2, U$3.1
- net GND: now also U$3.1; no longer Q1.3
- net GPIO15: no longer Q1.1
- net GPIO16: now also CHEAPO-2.3
- net GPIO4: now also U$3.2; no longer CHEAPO-2.3
- net VIN: no longer U$3.2
Routing:
- net GPIO15: track 124.4 -> 47.8 mm, vias 2 -> 0
- net VIN: track 206.2 -> 173.0 mm
- net GPIO4: track 54.0 -> 86.0 mm, vias 0 -> 1
- net N$5: track 101.4 -> 74.2 mm, vias 4 -> 2
- net GPIO16: track 56.2 -> 31.2 mm, vias 2 -> 1
- net GND: track 14.9 -> 0.00 mm, vias 38 -> 33
- net 3.3V: track 68.1 -> 81.7 mm, vias 2 -> 1
- net TX: track 60.6 -> 48.9 mm
- net RX: track 56.8 -> 47.0 mm
- net N$18: track 7.55 -> 0.00 mm, vias 1 -> 0
- net VFTDI: track 18.4 -> 23.6 mm, vias 1 -> 0
- net N$3: track 10.9 -> 16.0 mm, vias 2 -> 0
- net GPIO14: track 18.3 -> 22.3 mm, vias 2 -> 1
- net GPIO0: track 78.3 -> 74.6 mm, vias 1 -> 0
- net N$16: track 10.6 -> 14.2 mm
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